File: Kicad files/BACK_UP/ADACUS/ADACUS.kicad_pcb (KiCad board)
At the start: 4 copper layers, 68.6 x 88.9 mm, 115 parts, among them J200 USB_C_Receptacle_USB2.0_14P, U100 HT7533-1, U101 TLV62569DBV, U102 MCP6001-E/OT, U200 STM32F103CBT6, U201 USBLC6-2SC6, U301 REF3033, U302 MCP6001UT-E/OT, U303 MCP6001UT-E/OT, U401 MCP6001UT-E/OT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

Commit message: [Doc] File Import
Parts:
- D201, D202, D203, D204, D205: value PESD3V3L1UB,115 -> PESD3V3L1UB,115
- J200: footprint Connector_USB:USB_C_Receptacle_GCT_USB4105-xx-A_16P_TopMnt_Horizontal -> Connector_USB:USB_C_Receptacle_HRO_TYPE-C-31-M-12
- moved J200 3.16 mm to (179.6, 71.6)
- moved R203 1.17 mm to (144.9, 79.0), turned to 180 degrees
- moved R301 0.99 mm to (140.5, 83.9), turned to 0 degrees
- moved C203 0.61 mm to (151.0, 77.9)
- moved J400 0.39 mm to (163.1, 120.4)
- moved C108 0.06 mm to (146.0, 104.0)
Connections:
- U200 pad 20: unconnected-(U200-PB2-Pad20) -> DAC_NCLR
- U200 pad 21: DAC_NCLR -> DAC_NLDAC
- U200 pad 22: DAC_NLDAC -> unconnected-(U200-PB11-Pad22)
Routing:
- net +3V3: track 16.3 -> 151.9 mm, vias 0 -> 8
- net +5V: track 1.66 -> 86.0 mm, vias 0 -> 6
- net +3.3VA: track 9.39 -> 66.3 mm, vias 0 -> 5
- net VBUS: track 1.67 -> 35.8 mm, vias 0 -> 4
- net DAC_NLDAC: track 0.00 -> 27.2 mm, vias 0 -> 2
- net DAC_NCLR: track 0.00 -> 27.2 mm, vias 0 -> 2
- net VCOM: track 0.00 -> 26.8 mm, vias 0 -> 2
- net SPI2_MOSI: track 0.00 -> 22.9 mm, vias 0 -> 2
- net /MCU/MCU_NRST: track 0.00 -> 22.7 mm, vias 0 -> 2
- net /MCU/TIM4_CH2: track 0.00 -> 22.6 mm, vias 0 -> 2
- net /MCU/TIM4_CH1: track 0.00 -> 21.9 mm, vias 0 -> 2
- net SPI2_NSS: track 0.00 -> 20.4 mm, vias 0 -> 2
- net SPI2_SCK: track 0.00 -> 19.1 mm
- net SPI1_MISO: track 0.00 -> 18.8 mm
- net /MCU/TIM4_CH3: track 0.00 -> 18.8 mm, vias 0 -> 2
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- added copper zone on F.Cu, net /POWER/SW_BUCK
- added copper zone on In1.Cu, net GND
- added copper zone on In2.Cu, net GND
- removed copper zone on In1.Cu, net (none)
- removed copper zone on In2.Cu, net (none)
Other:
- board text added: "1 MOhm"
- board text added: "16/08/2024"
- board text added: "20Hz < BW < 20kHz"
- board text added: "50 Ohm"
- board text added: "ADACUS"
- board text added: "Author: A.B"
- board text added: "IN"
- board text added: "ON"
- board text added: "OUT"
- board text added: "USB"
