File: Kicad files/BACK_UP/ADACUS/ADC_ADACUS_sch.kicad_sch (KiCad schematic)
At the start: 32 parts, among them U301 REF3033, U302 MCP6001UT-E/OT, U303 MCP6001UT-E/OT

Commit message: [FILE] Finished board
Added PCB documents and finished schematics. Project is now done with both Altium and Kicad files uploaded
Parts:
- D300: value PESD3V3L1UB,115 -> PESD3V3L1UB,115
Changed lines of the file:
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@@
 			)
 		)
-		(property "Value" "PESD3V3L1UB,115 "
+		(property "Value" "PESD3V3L1UB,115"
 			(at 38.1 81.28 90)
 			(effects
