File: Kicad files/BACK_UP/ADACUS/DAC_ADACUS_sch.kicad_sch (KiCad schematic)
At the start: 17 parts, among them U401 MCP6001UT-E/OT

Commit message: [FILE] Finished board
Added PCB documents and finished schematics. Project is now done with both Altium and Kicad files uploaded
Parts:
- D400: value PESD3V3L1UB,115 -> PESD3V3L1UB,115
Changed lines of the file:
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@@
 			)
 		)
-		(property "Value" "PESD3V3L1UB,115 "
+		(property "Value" "PESD3V3L1UB,115"
 			(at 251.46 109.22 0)
 			(effects
