File: Kicad files/DAC_ADACUS_sch.kicad_sch (KiCad schematic)
At the start: 17 parts, among them U401 MCP6001UT-E/OT

Commit message: [FILE] Finished board
Added PCB documents and finished schematics. Project is now done with both Altium and Kicad files uploaded
Parts:
- C400, C402: footprint (none) -> Capacitor_SMD:C_0603_1608Metric
- C401, C403, C404, C405, C406: footprint (none) -> Capacitor_SMD:C_0402_1005Metric
- D400: value PESD3V3L1UB,115 -> PESD3V3L1UB,115; footprint (none) -> Diode_SMD:D_SOD-523
- J400: footprint (none) -> Connector_Coaxial:BNC_Amphenol_B6252HB-NPP3G-50_Horizontal
- R400, R401, R402, R403, R404, R405: footprint (none) -> Resistor_SMD:R_0402_1005Metric
- U400: footprint (none) -> Package_SO:VSSOP-10_3x3mm_P0.5mm
Other:
- company: (none) -> Head-Pin (TS)
- title: (none) -> DAC Schematic
- moved on the sheet: C400, C401, C402, C403, C404, C405, C406, D400, R400, R401, R402, R403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
