File: Kicad files/MCU_ADACUS_sch.kicad_sch (KiCad schematic)
At the start: 41 parts, among them J200 USB_C_Receptacle_USB2.0_14P, U200 STM32F103CBT6, U201 USBLC6-2SC6, Y200 16MHz

Commit message: [FILE] Finished board
Added PCB documents and finished schematics. Project is now done with both Altium and Kicad files uploaded
Parts:
- removed D200: ASMB-MTB1-0A3A2, LED_SMD:LED_Avago_PLCC4_3.2x2.8mm_CW, symbol LED:ASMB-MTB1-0A3A2
- removed J201: ~, symbol Connector:Conn_SWD_2x5_ADACUS
- added D200: ASMB-MTB0-0A3A2, LED_SMD:LED_RGB_Wuerth-PLCC4_3.2x2.8mm_150141M173100, symbol LED:ASMB-MTB0-0A3A2
- added J201: ~, Connector_PinHeader_1.27mm:PinHeader_2x05_P1.27mm_Vertical_SMD, symbol Adacus_lib:JST_CONN_ADACUS_2x5_1.27mm
- C200, C206, C207: footprint (none) -> Capacitor_SMD:C_0603_1608Metric
- C201, C202, C203, C204, C205, C208, C209, C210, C211, C212, C213: footprint (none) -> Capacitor_SMD:C_0402_1005Metric
- D201, D202, D203, D204, D205: value PESD3V3L1UB,115 -> PESD3V3L1UB,115; footprint (none) -> Diode_SMD:D_SOD-523
- J200: footprint (none) -> Connector_USB:USB_C_Receptacle_HRO_TYPE-C-31-M-12
- L200: footprint (none) -> Inductor_SMD:L_0402_1005Metric
- R200, R201, R202, R203, R204, R205, R206, R207, R208, R209, R210, R211, R212, R213: footprint (none) -> Resistor_SMD:R_0402_1005Metric
- Y200: footprint (none) -> Crystal:Crystal_SMD_2016-4Pin_2.0x1.6mm
Connections:
- net +3V3: now also D200.1 (A), J201.1
- net BLUE: now also D200.2 (BK)
- net DAC_NCLR: now also U200.20 (PB2); no longer U200.21 (PB10)
- net DAC_NLDAC: now also U200.21 (PB10); no longer U200.22 (PB11)
- net GND: now also J201.2, J201.3, J201.5
- net GREEN: now also D200.3 (GK)
- net R205_P10: now also J201.4
- net R206_P9: now also J201.6
- net R207_P8: now also J201.8
- net R208_P16: now also J201.9
- net RED: now also D200.4 (RK)
- net USB_CMC_D+: now also FL200.1; no longer FL200.4
- net USB_CMC_D-: now also FL200.4; no longer FL200.1
- net USB_CONN_D+: now also U201.4 (I/O2)
- net USB_CONN_D-: no longer U201.4 (I/O2)
- net USB_D+: now also FL200.2; no longer FL200.3
- net USB_D-: now also FL200.3; no longer FL200.2
- net XTAL_IN: now reaches C209.1, R201.1, Y200.3
- no-connect marks 20 -> 21
