File: Kicad files/Power_adacus_sch.kicad_sch (KiCad schematic)
At the start: 25 parts, among them U100 HT7533-1, U101 TLV62569DBV, U102 MCP6001-E/OT

Commit message: [FILE] Finished board
Added PCB documents and finished schematics. Project is now done with both Altium and Kicad files uploaded
Parts:
- C100, C101, C102, C103, C104, C105, C107: footprint (none) -> Capacitor_SMD:C_0603_1608Metric
- C106, C108: footprint (none) -> Capacitor_SMD:C_0402_1005Metric
- D100: renamed from D1; footprint (none) -> Diode_SMD:D_0402_1005Metric_Pad0.77x0.64mm_HandSolder
- H100, H101, H102, H103: footprint (none) -> MountingHole:MountingHole_2.7mm
- L100: footprint (none) -> Inductor_SMD:L_0402_1005Metric
- L101: footprint (none) -> Inductor_SMD:L_Cenker_CKCS4020
- R100, R101, R102, R103, R104, R105: footprint (none) -> Resistor_SMD:R_0402_1005Metric
Connections:
- net FB_BUCK: no longer R103.2
- net GND: now also R103.2
Other:
- moved on the sheet: C100, C101, C102, C103, C104, C105, C106, C107, C108, D100, H100, H101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
